File: USB2DXL/USB2DXL.kicad_pcb (KiCad board)
At the start: 4 copper layers, 38 x 42 mm, 43 parts, among them J1 XT60, J2 USB_C_Receptacle_USB2.0_16P, J3 Conn_01x03, J4 Conn_01x04, J5 Conn_01x03, J6 Conn_01x04, J7 Conn_01x04, U1 CH340E, U2 ISO7741DWR, U3 78L05G-AB3-R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

Commit message: パターンを引いた
Routing:
- net GNDPWR: track 24.5 -> 24.8 mm, vias 9 -> 27
- net GND: vias 9 -> 12
- added copper zone on B.Cu, net GND
- added copper zone on F.Cu, net GND
- added copper zone on B.Cu, net GNDPWR
- added copper zone on F.Cu, net GNDPWR

Commit message: pdfの追加
Routing:
- net GNDPWR: vias 27 -> 28
Changed lines of the file:
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@@
+	)
+	(via
+		(at 75.2348 93.4212)
+		(size 0.6)
+		(drill 0.3)
+		(layers "F.Cu" "B.Cu")
+		(free yes)
+		(net 5)
 	)
 	(via
